File: CAN_Debugger.kicad/CAN_Debugger.kicad_pcb (KiCad board)
At the start: 2 copper layers, 116 parts, among them J1 Conn_01x02, J15 RS-485, J16 RS-485, J2 Conn_01x04_MountingPin, J4 Conn_01x16_Socket, J5 USB_C_Receptacle_USB2.0, J6 RS-485, J7 CAN, J8 CAN, J9 CAN, Q1 AO3400A, SW1 SW_Push, SW2 SW_Push, SW3 SW_Push, U1 SN75176AD, U10 RS3236, U13 SN74LVC1G14DBV, U2 RY8411, U3 RS3236, U5 SIT1042T/3, U6 IP4220CZ6, U7 INA186, U8 STM32G431CBUx, U9 CH343P, Y1 25MHz

Commit message: update sche
Parts:
- removed D14: D, Diode_SMD:D_SMF
- added BZ1: Buzzer, 0_RM2023:MLT-9032, F.Cu at (131.3, 250.2)
- added C15: 1uf, Capacitor_SMD:C_0603_1608Metric, F.Cu at (178.6, 54.5)
- added C16: 1uf, Capacitor_SMD:C_0603_1608Metric, F.Cu at (178.6, 57.0)
- added C17: 2.2uf, Capacitor_SMD:C_0603_1608Metric, F.Cu at (178.6, 59.5)
- added C18: C, Capacitor_SMD:C_0603_1608Metric, F.Cu at (36.1, 81.8)
- added C19: C, Capacitor_SMD:C_0603_1608Metric, F.Cu at (36.1, 84.3)
- added C38: 100n, Capacitor_SMD:C_0603_1608Metric, F.Cu at (74.7, 117.6)
- added C39: C, Capacitor_SMD:C_0603_1608Metric, F.Cu at (72.6, 117.6)
- added C41: 100n, Capacitor_SMD:C_0603_1608Metric, F.Cu at (66.5, 117.7)
- added C46: C, Capacitor_SMD:C_0603_1608Metric, F.Cu at (76.6, 137.7)
- added C47: C, Capacitor_SMD:C_0603_1608Metric, F.Cu at (182.6, 57.0)
- added C51: 22u, Capacitor_SMD:C_1206_3216Metric_Pad1.33x1.80mm_HandSolder, F.Cu at (97.6, 228.3)
- added D10: D_Schottky, Diode_SMD:D_SMF, F.Cu at (102.2, 224.6)
- added F1: Fuse, Fuse:Fuse_1210_3225Metric_Pad1.42x2.65mm_HandSolder, B.Cu at (35.8, 141.5)
- added H1: MountingHole_Pad, MountingHole:MountingHole_2.2mm_M2_Pad_Via, F.Cu at (255.2, 120.2)
- added H2: MountingHole_Pad, MountingHole:MountingHole_2.2mm_M2_Pad_Via, F.Cu at (255.2, 126.1)
- added H3: MountingHole_Pad, MountingHole:MountingHole_2.2mm_M2_Pad_Via, F.Cu at (255.2, 132.1)
- added H4: MountingHole_Pad, MountingHole:MountingHole_2.2mm_M2_Pad_Via, F.Cu at (255.2, 138.0)
- added J3: Conn_01x02, Connector_AMASS:AMASS_XT30U-F_1x02_P5.0mm_Vertical, F.Cu at (95.2, 130.1)
- added L2: 4.7u, Inductor_SMD:L_0603_1608Metric, F.Cu at (100.4, 219.0)
- added R14: R, Resistor_SMD:R_0603_1608Metric, F.Cu at (182.6, 64.5)
- added R15: R, Resistor_SMD:R_0603_1608Metric, F.Cu at (40.1, 86.8)
- added R16: R, Resistor_SMD:R_0603_1608Metric, F.Cu at (38.7, 93.5)
- added R17: R, Resistor_SMD:R_0603_1608Metric_Pad0.98x0.95mm_HandSolder, F.Cu at (44.3, 94.3)
- added R24: R, Resistor_SMD:R_0603_1608Metric_Pad0.98x0.95mm_HandSolder, F.Cu at (44.3, 96.8)
- added R25: 33R, Resistor_SMD:R_0603_1608Metric_Pad0.98x0.95mm_HandSolder, F.Cu at (39.0, 90.7)
- added R26: 33R, Resistor_SMD:R_0603_1608Metric_Pad0.98x0.95mm_HandSolder, F.Cu at (44.3, 101.8)
- added R31: 10k, Resistor_SMD:R_0603_1608Metric_Pad0.98x0.95mm_HandSolder, F.Cu at (71.1, 117.6)
- added R38: 10k, Resistor_SMD:R_0603_1608Metric, F.Cu at (68.9, 118.5)
- added R39: 10k, Resistor_SMD:R_0603_1608Metric, F.Cu at (78.7, 118.5)
- added R4: R, Resistor_SMD:R_2512_6332Metric, B.Cu at (60.8, 147.3)
- added R40: 10k, Resistor_SMD:R_0603_1608Metric, F.Cu at (70.3, 137.7)
- added R41: 100k, Resistor_SMD:R_0603_1608Metric, F.Cu at (76.7, 139.2)
- added R42: 10k, Resistor_SMD:R_0603_1608Metric, F.Cu at (65.8, 131.3)
- added R43: R, Resistor_SMD:R_0603_1608Metric, F.Cu at (44.1, 84.3)
- added R44: R, Resistor_SMD:R_2512_6332Metric, F.Cu at (86.5, 136.1)
- added R45: R, Resistor_SMD:R_0603_1608Metric, F.Cu at (89.1, 129.3)
- added R48: 100k, Resistor_SMD:R_0603_1608Metric, F.Cu at (186.6, 69.5)
- added R49: R, Resistor_SMD:R_0603_1608Metric, F.Cu at (186.6, 72.0)
- added R51: R, Resistor_SMD:R_0603_1608Metric, F.Cu at (88.3, 132.6)
- added R52: 100k, Resistor_SMD:R_0603_1608Metric, F.Cu at (190.6, 57.0)
- added R6: 10k, Resistor_SMD:R_0603_1608Metric_Pad0.98x0.95mm_HandSolder, F.Cu at (76.5, 117.6)
- added R61: 19k, Resistor_SMD:R_0603_1608Metric, F.Cu at (102.4, 232.2)
- added R62: 1k, Resistor_SMD:R_0603_1608Metric, F.Cu at (102.4, 234.7)
- added SW4: RotaryEncoder_Switch, Rotary_Encoder:RotaryEncoder_Alps_EC11E-Switch_Vertical_H20mm, F.Cu at (76.2, 120.8)
- added U4: GS8332-SR, Package_SO:MSOP-8_3x3mm_P0.65mm, F.Cu at (44.0, 91.7)
- C104, C105, C34, C40, C42, D1, R59, R60, U7: moved to B.Cu
- C48: value 100n -> 22u; footprint Capacitor_SMD:C_0603_1608Metric -> Inductor_SMD:L_0603_1608Metric
- R50: value 33k -> 10k
- U13: value SN74LVC1G14DBV -> MT3608; footprint Package_TO_SOT_SMD:SOT-23-5 -> Package_TO_SOT_SMD:SOT-23-6
- moved C37 208.3 mm to (-66.8, 85.9)
- moved C45 208.3 mm to (-66.8, 89.2)
- moved F4 208.3 mm to (-60.5, 90.1)
- moved U9 208.3 mm to (-54.4, 90.2)
- moved C20 196.8 mm to (-81.3, 96.7)
- moved C21 196.8 mm to (-81.3, 99.2)
- moved C36 196.8 mm to (-73.3, 76.6)
- moved C43 196.8 mm to (-73.3, 84.2)
- moved C44 196.8 mm to (-73.3, 86.7)
- moved D4 196.8 mm to (-61.6, 104.3)
- moved D6 196.8 mm to (-33.7, 84.6)
- moved FB1 196.8 mm to (-73.3, 101.7)
- moved R32 196.8 mm to (-65.3, 96.7)
- moved R33 196.8 mm to (-65.3, 99.2)
- moved R34 196.8 mm to (-65.3, 101.7)
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Connections:
- net IA+ renamed +24V
- C1 pad 2: VSS -> GND
- C10 pad 2: VSS -> GND
- C104 pad 1: VSS -> GND
- C105 pad 2: VSS -> GND
- C11 pad 2: VSS -> GND
- C12 pad 1: VDD -> +3.3V
- C12 pad 2: VSS -> GND
- C13 pad 1: VDD -> +3.3V
- C13 pad 2: VSS -> GND
- C14 pad 2: VSS -> GND
- C2 pad 2: VSS -> GND
- C20 pad 2: VSS -> GND
- C21 pad 2: VSS -> GND
- C22 pad 1: VSS -> GND
- C22 pad 2: VBAT -> +5V
- C23 pad 2: VBAT -> +5V
- C24 pad 1: VSS -> GND
- C24 pad 2: VBAT -> +5V
- C25 pad 1: VDD -> +3.3V
- C25 pad 2: VSS -> GND
- C26 pad 1: VDD -> +3.3V
- C26 pad 2: VSS -> GND
- C27 pad 1: VDD -> +3.3V
- C27 pad 2: VSS -> GND
- C28 pad 1: VDD -> +3.3V
- C28 pad 2: VSS -> GND
- C29 pad 1: VDD -> +3.3V
- C29 pad 2: VSS -> GND
- C3 pad 2: VSS -> GND
- C30 pad 1: VDD -> +3.3V
- C30 pad 2: VSS -> GND
- C31 pad 1: VSS -> GND
- C32 pad 1: VSS -> GND
- C33 pad 1: VSS -> GND
- C35 pad 1: VSS -> GND
- C36 pad 2: VSS -> GND
- C37 pad 2: VSS -> GND
- C40 pad 1: /1.65Vref -> PB1
- C40 pad 2: VSS -> GND
- C42 pad 1: +3.3VA -> +3.3V
- C42 pad 2: VSS -> GND
- C43 pad 1: VSS -> GND
- C44 pad 2: VSS -> GND
- C45 pad 2: VSS -> GND
- C48 pad 1: Net-(D14-A) -> VCC
- C48 pad 2: VSS -> GND
- C49 pad 1: VBAT -> +5V
- C49 pad 2: VSS -> GND
- C50 pad 1: VBAT -> +5V
- C50 pad 2: VSS -> GND
- C6 pad 2: VSS -> GND
- C7 pad 2: VSS -> GND
- C8 pad 2: VSS -> GND
- C9 pad 2: VSS -> GND
- D1 pad 2: VSS -> GND
- D2 pad 1: VBAT -> +5V
- D3 pad 2: VBAT -> +5V
- D4 pad 1: VSS -> GND
- D5 pad 1: VBAT -> +5V
- D7 pad 1: VDD -> +3.3V
- D7 pad 2: VSS -> GND
- D8 pad 3: VSS -> GND
- F2 pad 1: VDD -> +3.3V
- J1 pad 1: VSS -> GND
- J15 pad MP: VSS -> GND
- J16 pad MP: VSS -> GND
- J2 pad 3: VSS -> GND
- J2 pad MP: VSS -> GND
- J4 pad 16: VSS -> GND
- J4 pad 5: VBAT -> +5V
- J4 pad 7: VDD -> +3.3V
- J5 pad A1: VSS -> GND
- J5 pad A12: VSS -> GND
- J5 pad B1: VSS -> GND
- J5 pad B12: VSS -> GND
- J6 pad MP: VSS -> GND
- J7 pad MP: VSS -> GND
- J8 pad MP: VSS -> GND
- J9 pad MP: VSS -> GND
- Q1 pad 2: VSS -> GND
- R10 pad 1: VSS -> GND
- R19 pad 1: VDD -> +3.3V
- R21 pad 1: VDD -> +3.3V
- R23 pad 1: VDD -> +3.3V
- R28 pad 2: VSS -> GND
- R3 pad 2: VSS -> GND
- R30 pad 2: VSS -> GND
- R34 pad 1: VSS -> GND
- R35 pad 1: VSS -> GND
- R37 pad 1: VSS -> GND
- R50 pad 1: Net-(U1-D) -> +5V
- R50 pad 2: Net-(D14-A) -> Net-(U13-EN)
- R53 pad 1: MCU_3.3V -> +3.3V
- R54 pad 2: RS485_TX -> PB10
- R55 pad 1: RS485_RX -> PB11
- R56 pad 1: VSS -> GND
- R58 pad 2: VBAT -> +5V
- SW1 pad 2: VSS -> GND
- SW2 pad 2: VSS -> GND
- SW3 pad 2: VSS -> GND
- U1 pad 2: RX485_DE -> PB14
- U1 pad 3: RX485_DE -> PB14
- U1 pad 5: VSS -> GND
- U1 pad 8: VBAT -> +5V
- U10 pad 2: VSS -> GND
- U13 pad 1: unconnected-(U13-NC-Pad1) -> Net-(D10-A)
- U13 pad 2: Net-(D14-A) -> GND
- U13 pad 3: VSS -> Net-(U13-FB)
- U13 pad 4: RX485_DE -> Net-(U13-EN)
- U13 pad 5: VBAT -> +5V
- U2 pad 2: VSS -> GND
- U3 pad 2: VSS -> GND
- U3 pad 5: VDD -> +3.3V
- U5 pad 2: VSS -> GND
- U5 pad 3: VBAT -> +5V
- U5 pad 5: VDD -> +3.3V
- U6 pad 2: VSS -> GND
- U7 pad 2: VSS -> GND
- U7 pad 3: +3.3VA -> +3.3V
- U8 pad 1: VDD -> +3.3V
- U8 pad 21: VDD -> +3.3V
- U8 pad 23: VDD -> +3.3V
- U8 pad 32: PA10 -> Encoder_button
- U8 pad 35: VDD -> +3.3V
- U8 pad 38: PA15 -> CS
- U8 pad 48: VDD -> +3.3V
- U8 pad 49: VSS -> GND
- U9 pad 17: VSS -> GND
- U9 pad 2: VSS -> GND
Other:
- copper layers 2 -> 4

Commit message: update schematic
Parts:
- removed C18, C19: C, Capacitor_SMD:C_0603_1608Metric
- removed C32: 100n, Capacitor_SMD:C_0603_1608Metric
- removed D2: D_Schottky, Diode_SMD:D_SMF
- removed R16, R43, R49: R, Resistor_SMD:R_0603_1608Metric
- removed R17, R24: R, Resistor_SMD:R_0603_1608Metric_Pad0.98x0.95mm_HandSolder
- removed R20: 330, Resistor_SMD:R_0603_1608Metric
- removed R21: 10k, Resistor_SMD:R_0603_1608Metric
- removed R25, R26: 33R, Resistor_SMD:R_0603_1608Metric_Pad0.98x0.95mm_HandSolder
- removed SW2: SW_Push, Button_Switch_SMD:SW_SPST_TL3342
- removed U4: GS8332-SR, Package_SO:MSOP-8_3x3mm_P0.65mm
- added D11: D_Schottky, Diode_SMD:D_SMF, F.Cu at (28.9, 128.6)
- added D9: LED, LED_SMD:LED_0603_1608Metric, F.Cu at (31.0, 118.1)
- C15, C16, C17, C20, C21, C35, C36, C37, C43, C44, C45, D6, F4, FB1, J4, J5, R14, R27, R28, R34, R35, R37, R5, U10, U6, U9: moved to B.Cu
- C48: footprint Inductor_SMD:L_0603_1608Metric -> Capacitor_SMD:C_1206_3216Metric
- L1: footprint Inductor_SMD:L_Bourns-SRN4018 -> Inductor_SMD:L_Sunlord_MWSA0402S
- L2: footprint Inductor_SMD:L_0603_1608Metric -> Inductor_SMD:L_Sunlord_MWSA0402S
- Y1: footprint Crystal:Crystal_SMD_5032-2Pin_5.0x3.2mm -> Crystal:Crystal_SMD_3225-4Pin_3.2x2.5mm
- moved J2 247.6 mm to (59.5, 86.1), turned to 180 degrees
- moved F2 243.8 mm to (56.0, 92.3), turned to 90 degrees
- moved D7 238.4 mm to (58.5, 92.3)
- moved R13 231.9 mm to (61.6, 99.6), turned to 90 degrees
- moved R12 231.6 mm to (60.0, 99.6), turned to 90 degrees
- moved R61 149.6 mm to (45.8, 93.8), turned to -90 degrees
- moved R62 149.5 mm to (44.7, 96.8), turned to -90 degrees
- moved C48 149.5 mm to (48.4, 89.6)
- moved C15 149.3 mm to (33.6, 90.1)
- moved C16 145.8 mm to (36.7, 90.2)
- moved R14 143.6 mm to (41.8, 92.4), turned to -90 degrees
- moved R50 142.5 mm to (47.4, 100.3), turned to 180 degrees
- moved D10 142.5 mm to (47.7, 92.9), turned to -90 degrees
- moved U13 142.0 mm to (47.2, 97.4), turned to -90 degrees
- moved R52 140.0 mm to (64.8, 118.4)
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Connections:
- C1 pad 1: Net-(D2-A) -> +5V
- C2 pad 1: Net-(D2-A) -> +5V
- C3 pad 1: Net-(D2-A) -> +5V
- C5 pad 1: Net-(D2-A) -> +5V
- H1 pad 1: GND -> unconnected-(H1-Pad1)
- H2 pad 1: GND -> unconnected-(H2-Pad1)
- H3 pad 1: GND -> unconnected-(H3-Pad1)
- H4 pad 1: GND -> unconnected-(H4-Pad1)
- L1 pad 2: Net-(D2-A) -> +5V
- R15 pad 2: ADC_1 -> Net-(D9-A)
- R2 pad 1: Net-(D2-A) -> +5V
- R48 pad 1: +3.3V -> +3.3VA
- U8 pad 11: ADC_2 -> PA3
- U8 pad 21: +3.3V -> +3.3VA
- U8 pad 9: ADC_1 -> PA1
- Y1 pad 2: RCC_OSC_IN -> GND

Commit message: Update PCB layout
Parts:
- removed D11: D_Schottky, Diode_SMD:D_SMF
- added C32: C, Capacitor_SMD:C_0603_1608Metric, B.Cu at (61.3, 136.7)
- added C52: C, Capacitor_SMD:C_0603_1608Metric, B.Cu at (59.7, 135.2)
- added C53: C, Capacitor_SMD:C_0603_1608Metric, B.Cu at (64.3, 135.2)
- added C54: C, Capacitor_SMD:C_0603_1608Metric, B.Cu at (62.8, 136.7)
- added C57: 100n, Capacitor_SMD:C_0603_1608Metric, B.Cu at (71.2, 122.5)
- added C58: 100n, Capacitor_SMD:C_0603_1608Metric, B.Cu at (67.4, 126.1)
- added C59: 100n, Capacitor_SMD:C_0603_1608Metric, B.Cu at (76.0, 132.2)
- added C70: 100n, Capacitor_SMD:C_0603_1608Metric, B.Cu at (70.7, 132.5)
- added C76: 100n, Capacitor_SMD:C_0603_1608Metric, B.Cu at (63.5, 128.0)
- added C80: 10u, Capacitor_SMD:C_0603_1608Metric, B.Cu at (53.9, 134.6)
- added C88: 100n, Capacitor_SMD:C_0603_1608Metric, B.Cu at (66.6, 131.2)
- added JP1: SolderJumper_2_Open, Jumper:SolderJumper-2_P1.3mm_Open_TrianglePad1.0x1.5mm, B.Cu at (62.3, 122.2)
- added L3: L_Ferrite, Inductor_SMD:L_0603_1608Metric, B.Cu at (62.0, 134.4)
- added R16: 100k 25ppm, Resistor_SMD:R_0603_1608Metric, B.Cu at (73.7, 123.5)
- added R17: 100k 25ppm, Resistor_SMD:R_0603_1608Metric, B.Cu at (72.9, 121.2)
- added R20: 33r, Resistor_SMD:R_0603_1608Metric, B.Cu at (68.2, 123.8)
- added R21: 100k 25ppm, Resistor_SMD:R_0603_1608Metric, B.Cu at (73.7, 133.2)
- added R24: 1k, Resistor_SMD:R_0603_1608Metric, B.Cu at (66.7, 123.8)
- added R25: 10k 25ppm, Resistor_SMD:R_0603_1608Metric, B.Cu at (76.0, 130.6)
- added R63: 33r, Resistor_SMD:R_0603_1608Metric, B.Cu at (67.4, 128.9)
- added RN1: R_Pack04, Resistor_SMD:R_Array_Convex_4x0603, F.Cu at (49.7, 105.5)
- added U14: GS8332-SR, Package_SO:SOIC-8_3.9x4.9mm_P1.27mm, B.Cu at (71.7, 127.9)
- BZ1, C22, C23, C24, C29, C30, D5, Q1, R10, R11: moved to B.Cu
- C39, C46: value C -> 100n
- D1: value SMDJ28A -> SMCJ28A
- R57: value 120 -> 120r
- moved R10 71.8 mm to (64.0, 110.3), turned to 180 degrees
- moved Q1 70.1 mm to (67.5, 107.7)
- moved BZ1 56.7 mm to (72.9, 112.3), turned to -90 degrees
- moved C22 56.6 mm to (72.0, 118.5)
- moved R11 53.3 mm to (64.0, 108.7), turned to 0 degrees
- moved D5 53.0 mm to (81.9, 112.2), turned to 90 degrees
- moved C24 46.7 mm to (78.0, 115.8), turned to 180 degrees
- moved C23 46.6 mm to (79.8, 112.2), turned to -90 degrees
- moved J16 27.6 mm to (79.4, 119.8), turned to 0 degrees
- moved C50 27.5 mm to (77.8, 141.3), turned to -90 degrees
- moved J15 27.1 mm to (79.4, 126.2), turned to 0 degrees
- moved J6 26.7 mm to (79.4, 132.8), turned to 0 degrees
- moved D8 24.6 mm to (75.9, 137.8)
- moved R57 24.1 mm to (79.4, 136.9), turned to 0 degrees
- moved C46 23.0 mm to (82.8, 109.1)
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Connections:
- C14 pad 1: RCC_OSC_OUT -> RCC_OSC_IN
- C29 pad 1: +3.3V -> +3.3VA
- C30 pad 1: +3.3V -> +3.3VA
- C40 pad 1: PB1 -> /1.65Vref
- C8 pad 1: RCC_OSC_IN -> RCC_OSC_OUT
- D9 pad 1: CANL -> CANH
- R15 pad 1: CANH -> CANL
- R32 pad 1: Net-(U9-RXD) -> PB6
- R32 pad 2: PB6 -> Net-(U9-RXD)
- R39 pad 1: +3.3V -> Net-(R39-Pad1)
- R39 pad 2: Net-(R39-Pad2) -> +3.3V
- R6 pad 2: Net-(R39-Pad2) -> Net-(R39-Pad1)
- SW4 pad A: Net-(R39-Pad2) -> Net-(R39-Pad1)
- U7 pad 1: PB1 -> /1.65Vref
- U8 pad 29: PC6 -> BUZZER
- U8 pad 38: CS -> PA15
- U8 pad 40: D/C -> PC11
- U8 pad 41: SCLK -> SPI1_SCK
- U8 pad 43: SDIN -> SPI1_MOSI
- Y1 pad 1: RCC_OSC_OUT -> RCC_OSC_IN
- Y1 pad 3: RCC_OSC_IN -> RCC_OSC_OUT
Routing:
- net SDIN: track 0.00 -> 33.7 mm, vias 0 -> 1
- net PA7: track 0.00 -> 31.6 mm
- net A+: track 0.00 -> 30.8 mm
- net Net-(C46-Pad1): track 0.00 -> 29.7 mm
- net +3.3V: track 0.00 -> 29.6 mm, vias 0 -> 38
- net PC10: track 0.00 -> 28.6 mm, vias 0 -> 3
- net B-: track 0.00 -> 27.8 mm
- net PB14: track 0.00 -> 27.7 mm
- net CANH: track 0.00 -> 26.6 mm
- net D/C: track 0.00 -> 26.4 mm, vias 0 -> 1
- net VBUS_USBTTL: track 0.00 -> 25.9 mm, vias 0 -> 3
- net CANL: track 0.00 -> 25.3 mm
- net USB_UART_DM: track 0.00 -> 25.0 mm, vias 0 -> 2
- net A_I: track 0.00 -> 24.6 mm, vias 0 -> 1
- net +5V: track 0.00 -> 23.6 mm, vias 0 -> 28
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- added copper zone on B.Cu, net +24V
- added copper zone on F.Cu, net +24V
- added copper zone on In2.Cu, net +24V
- added copper zone on F.Cu, net +3.3V
- added copper zone on In2.Cu, net +3.3V
- added copper zone on B.Cu, net +3.3VA
- added copper zone on In2.Cu, net +3.3VA
- added copper zone on In2.Cu, net +3.3V_USBTTL
- added copper zone on F.Cu, net +5V
- added copper zone on In2.Cu, net +5V
- added copper zone on B.Cu, net /1.65Vref
- added copper zone on In2.Cu, net /1.65Vref
- added copper zone on B.Cu, net /VBUS_CONNECTOR
- added copper zone on In2.Cu, net /VBUS_CONNECTOR
- added copper zone on B.Cu, net 24v_motor
- added copper zone on B.Cu, net GND
- added copper zone on F.Cu, net GND
- added copper zone on In1.Cu, net GND
- added copper zone on F.Cu, net Net-(D10-A)
- added copper zone on F.Cu, net Net-(D3-K)
- added copper zone on F.Cu, net Net-(U2-LX)
- added copper zone on B.Cu, net VBUS_USBTTL
- added copper zone on B.Cu, net VCC
- added copper zone on F.Cu, net VCC
- added copper zone on F.Cu, net iA+
Other:
- board outline added: 59.4 x 76.4 mm
