File: CAN_Debugger.kicad/CAN_Debugger.kicad_sch (KiCad schematic)
At the start: 72 parts, among them J1 Conn_01x02, J2 Conn_01x04_MountingPin, J4 Conn_01x16_Socket, J7 CAN, J8 CAN, J9 CAN, Q1 AO3400A, SW1 SW_Push, SW2 SW_Push, SW3 SW_Push, U1 STM32F103C8Tx, U2 RY8411, U3 RS3236, U5 TJA1042T-3, Y1 Crystal

Commit message: Kicad Schematic done
Parts:
- removed R5: 330, symbol Device:R
- added C104, C105, C34, C35, C38, C39, C40, C41, C42: 100n, Capacitor_SMD:C_0603_1608Metric, symbol Device:C
- added C18, C19: C, symbol Device:C
- added D10: D_Schottky, Diode_SMD:D_SMF, symbol Device:D_Schottky
- added F3: Fuse, Fuse:Fuse_1206_3216Metric, symbol Device:Fuse
- added J13: Conn_01x04, ENTERPRIZE2024_internal_JYC_v0:Micro USB, symbol Connector_Generic:Conn_01x04
- added R15, R16, R17, R24, R4: R, symbol Device:R
- added R25, R26: 33R, symbol Device:R
- added R27, R29: 330, Resistor_SMD:R_0603_1608Metric, symbol Device:R
- added R28: 10k, Resistor_SMD:R_0603_1608Metric, symbol Device:R
- added R30, R31: 33, Resistor_SMD:R_0603_1608Metric, symbol Device:R
- added R59, R60: 100r 25ppm, Resistor_SMD:R_0603_1608Metric, symbol Device:R
- added SW4: SW_Push, Button_Switch_SMD:SW_SPST_TL3342, symbol Switch:SW_Push
- added U4: GS8332-SR, symbol 0_RM2023:GS8332-SR
- added U7: INA186, Package_TO_SOT_SMD:SOT-363_SC-70-6, symbol Amplifier_Current:INA199xxDCK
- added U8: ch343p, ENTERPRIZE2024_internal_JYC_v0:QFN17, symbol 0_RM2023:ch343p
- Y1: value Crystal -> 8MHz
Connections:
- net PA8 is gone; now on net CS: U1.29 (PA8)
- net SPI1_MOSI is gone; now on net SDIN: U1.17 (PA7)
- net SPI1_SCK is gone; now on net SCLK: U1.15 (PA5)
- net +24V: now also R4.1, R59.1
- net +3.3V: now also C38.1, C39.1, C41.1, R28.1, U4.8 (VDD), U8.1 (VIO), U8.3 (VDD5), U8.6 (V3)
- net +5V: now also D10.1 (K), R29.2
- net CANH: now also R15.1
- net CANL: now also R17.2
- net GND: now also C104.1, C105.2, C18.2, C19.2, C35.1, C38.2, C39.2, C40.2, C41.2, C42.2, J13.1 (Pin_1), R16.2, R24.2, SW4.2, U4.4 (VSS), U7.2 (GND), U8.17 (GND), U8.2 (GND)
- net RES: now also C35.2, R27.2
- net PA0 renamed A_I
- net A_I: now also U7.6
- net PA2 renamed ADC_1
- net ADC_1: now also R25.1
- net PA4 renamed ADC_2
- net ADC_2: now also R26.2
- new net: C104.2, C34.1, R59.2, U7.4 (+)
- new net: R27.1, R28.2, SW4.1
- new net: F3.1, J13.4 (Pin_4)
- new net: R31.1, U8.5 (RXD)
- new net: C19.1, R17.1, R24.1, U4.5 (+)
- new net: C18.1, R15.2, R16.1, U4.3 (+)
- new net: R25.2, U4.1 (OUTA), U4.2 (-)
- new net: R26.1, U4.6 (-), U4.7 (OUTB)
- new net: D10.2 (A), F3.2
- new net: C105.1, C34.2, R60.2, U7.5 (-)
- new net: R30.1, U8.4 (TXD)
- new net: R29.1, U8.9 (VBUS)
- new net +3.3VA: C42.1, U7.3 (V+)
- new net 1.65Vref: C40.1, U7.1 (REF)
- new net 24v_motor: R4.2, R60.1
- new net Mini-PC_D+: J13.2 (Pin_2), U8.7 (VD+)
- new net Mini-PC_D-: J13.3 (Pin_3), U8.8 (VD-)
- new net UART3_RX: R30.2
- new net UART3_TX: R31.2
- no-connect marks 0 -> 7
Other:
- moved on the sheet: C14, C25, C26, C27, C28, C29, C30, C31, C32, C33, C8, J4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

Commit message: Changing schematic; Change cubemx ioc to G431
Parts:
- removed C38, C39, C41: 100n, Capacitor_SMD:C_0603_1608Metric, symbol Device:C
- removed D10: D_Schottky, Diode_SMD:D_SMF, symbol Device:D_Schottky
- removed D2: SMF5V0A, Diode_SMD:D_SMF, symbol Diode:SMF5V0A
- removed F3: Fuse, Fuse:Fuse_1206_3216Metric, symbol Device:Fuse
- removed J13: Conn_01x04, ENTERPRIZE2024_internal_JYC_v0:Micro USB, symbol Connector_Generic:Conn_01x04
- removed R31: 33, Resistor_SMD:R_0603_1608Metric, symbol Device:R
- removed U8: ch343p, ENTERPRIZE2024_internal_JYC_v0:QFN17, symbol 0_RM2023:ch343p
- added C18, C21: 10nF, Capacitor_SMD:C_0603_1608Metric, symbol Device:C
- added C19, C20: 10uF, Capacitor_SMD:C_1206_3216Metric, symbol Device:C
- added C22, C23, C24: 100nF, Capacitor_SMD:C_0603_1608Metric, symbol Device:C
- added D2, D6: D_Schottky, Diode_SMD:D_SMF, symbol Device:D_Schottky
- added D27: LED, LED_SMD:LED_0603_1608Metric, symbol Device:LED
- added F2: Fuse, Fuse:Fuse_1812_4532Metric, symbol Device:Fuse
- added FB1: 120R@100MHz, Inductor_SMD:L_0603_1608Metric, symbol Device:FerriteBead
- added J4: USB_C_Receptacle_USB2.0, Connector_USB:USB_C_Receptacle_HRO_TYPE-C-31-M-12, symbol Connector:USB_C_Receptacle_USB2.0
- added R10, R11: 5.1k, Resistor_SMD:R_0603_1608Metric, symbol Device:R
- added R12: 1M, Resistor_SMD:R_0603_1608Metric, symbol Device:R
- added R13: 330R, Resistor_SMD:R_0603_1608Metric, symbol Device:R
- added R14, R15: 33R, Resistor_SMD:R_0603_1608Metric, symbol Device:R
- added R56: 10K, Resistor_SMD:R_0603_1608Metric, symbol Device:R
- added U4: CH343P, Package_DFN_QFN:TQFN-16-1EP_3x3mm_P0.5mm_EP1.23x1.23mm, symbol 0_RM2023:ch343p
- added U6: RS3236, Package_TO_SOT_SMD:SOT-23-5, symbol Regulator_Linear:LDK130-12_SOT23_SOT353
- added U7: IP4220CZ6, Package_TO_SOT_SMD:SOT-23-6, symbol Power_Protection:CDSOT236-0504C
- C1, C2, C6, C7: value C -> 10uF
- C3: value C_Polarized -> 47uF
- R29: value 330 -> 120R
- R30: value 33 -> 10K
- U5: value TJA1042T-3 -> SIT1042T/3
Connections:
- net +3.3V: no longer J4.5 (Pin_5)
- net +5V: now also J4.5 (Pin_5), D2.1 (K); no longer C1.1, C2.1, C3.1, C5.1, J4.15 (Pin_15), L1.2, R2.1, R29.2
- net GND: now also R30.2, C18.1, C19.2, C20.2, C21.2, C22.2, C23.2, C24.2, D27.1 (K), J4.A1 (GND), J4.A12 (GND), J4.B1 (GND), J4.B12 (GND), R10.1, R11.1, R12.1, U4.17 (GND), U4.2 (GND), U6.2 (GND), U7.2 (VN); no longer U5.8 (STB)
- net UART3_RX: now also R14.2; no longer R30.2
- net UART3_TX: now also R15.2
- net at U2.1 (BS): now also C4.1
- net CAN_STB: now reaches R30.1
- net CAN_STB: now also R29.1
- new net: C1.1, C2.1, C3.1, C5.1, D2.2 (A), L1.2, R2.1
- new net: C18.2, J4.S1 (SHIELD), R12.2
- new net: D27.2 (A), R56.2
- new net: R14.1, U4.4 (TXD)
- new net: R15.1, U4.5 (RXD)
- new net: J4.A5 (CC1), R10.2
- new net: D6.1 (K), F2.2
- new net: F2.1, FB1.2
- new net: J4.B5 (CC2), R11.2
- new net: C21.1, U6.4 (BP)
- new net: R13.1, U4.9 (VBUS)
- new net: R29.2, U5.8 (STB)
- new net +3.3V_USBTTL: C20.1, C22.1, C23.1, C24.1, U4.1 (VIO), U4.3 (VDD5), U4.6 (V3), U6.5 (OUT)
- new net USB_UART_DM: J4.A7 (D-), J4.B7 (D-), U4.8 (VD-), U7.6 (IO4)
- new net USB_UART_DP: J4.A6 (D+), J4.B6 (D+), U4.7 (VD+), U7.1 (IO1)
- new net VBUS_CONNECTOR: D6.2 (A), J4.A4 (VBUS), J4.A9 (VBUS), J4.B4 (VBUS), J4.B9 (VBUS)
- new net VBUS_USBTTL: C19.1, FB1.1, R13.2, R56.1, U6.1 (IN), U6.3 (EN), U7.5 (VP)
- new net VCC: J4.15 (Pin_15)
- no-connect marks 7 -> 11
Other:
- moved on the sheet: C1, C14, C2, C25, C26, C27, C28, C29, C3, C30, C31, C32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

Commit message: update sch
Parts:
- removed SW4: SW_Push, Button_Switch_SMD:SW_SPST_TL3342, symbol Switch:SW_Push
- removed U1: STM32F103C8Tx, Package_QFP:LQFP-48_7x7mm_P0.5mm, symbol MCU_ST_STM32F1:STM32F103C8Tx
- added C38, C41: 100n, symbol Device:C
- added C39, C46: C, symbol Device:C
- added J3: Conn_01x02, symbol Connector_Generic:Conn_01x02
- added R31, R38, R39, R40, R42: 10k, symbol Device:R
- added R41: 100k, symbol Device:R
- added R43, R44, R45, R46, R47, R48, R49, R50: R, symbol Device:R
- added SW4: RotaryEncoder_Switch, symbol Device:RotaryEncoder_Switch
- added U11: OPAMP2, Package_TO_SOT_SMD:TSOT-23-5, symbol Amplifier_Operational:AD8603
- added U12: OPAMP3, Package_TO_SOT_SMD:TSOT-23-5, symbol Amplifier_Operational:AD8603
- added U8: STM32G431CBUx, Package_DFN_QFN:QFN-48-1EP_7x7mm_P0.5mm_EP5.6x5.6mm, symbol MCU_ST_STM32G4:STM32G431CBUx
- R6: value 1k -> 10k; footprint Resistor_SMD:R_0603_1608Metric -> (none)
- Y1: value 8MHz -> 25MHz
Connections:
- net UART3_RX is gone; now on net PB7: R14.2
- net UART3_TX is gone; now on net PB6: R15.2
- net +3.3V: now also C41.1, R38.1, R39.1, R40.1, U8.1 (VBAT), U8.21 (VDDA), U8.23 (VDD), U8.35 (VDD), U8.48 (VDD); no longer R28.1
- net 24v_motor: now also J3.1 (Pin_1)
- net ADC_1: now also R15.2, U8.9 (PA1)
- net ADC_2: now also R43.2, U8.11 (PA3)
- net A_I: now also U8.8 (PA0)
- net CANH: now also C18.1, R16.1, U4.3 (+)
- net CANL: now also R43.1
- net CAN_RX: now also U8.46 (PB8)
- net CAN_STB: now also U8.2 (PC13)
- net CAN_TX: now also U8.47 (PB9)
- net D/C: now also U8.40 (PC11)
- net GND: now also R28.2, C38.1, C39.2, C41.2, C46.2, R41.2, R44.1, R48.2, SW4.C, U8.49 (VSS); no longer R6.1
- net NRST: now also U8.7 (PG10)
- net PA10: now also U8.32 (PA10)
- net PA15: now also U8.38 (PA15)
- net PA9: now also U8.31 (PA9)
- net PB0: now also R48.1, U12.3 (+), U8.17 (PB0)
- net PB1: now also R49.2, R50.1, R50.2, U12.1, U8.18 (PB1)
- net PB10: now also U8.22 (PB10)
- net PB11: now also U8.24 (PB11)
- net PB12: now also U8.25 (PB12)
- net PB13: now also U8.26 (PB13)
- net PB14: now also U8.27 (PB14)
- net PB15: now also U8.28 (PB15)
- net PB2: now also R49.1, U12.4 (-), U8.19 (PB2)
- net PB4: now also U8.42 (PB4)
- net PB6: now also U8.44 (PB6)
- net PB7: now also U8.45 (PB7)
- net PC14: now also U8.3 (PC14)
- net PC15: now also U8.4 (PC15)
- net RCC_OSC_IN: now also U8.5 (PF0)
- net RCC_OSC_OUT: now also U8.6 (PF1)
- net RES: now also R28.1
- net SCLK: now also U8.41 (PB3)
- net SDIN: now also U8.43 (PB5)
- net SYS_JTCK-SWDCLK: now also U8.37 (PA14)
- net SYS_JTMS-SWDIO: now also U8.36 (PA13)
- net PC10: now reaches R27.1
- net PC10: now also U8.39 (PC10); no longer R28.2
- net BOOT0: no longer names the net of R6.2
- net BOOT0: now also R39.2, SW4.A
- new net: R31.2, R38.2, SW4.B
- new net: C46.1, R41.1, R42.2, SW4.S2
- new net: R40.2, SW4.S1
- new net PA11: C39.1, R31.1, U8.33 (PA11)
- new net PA12: C38.2, R6.1, U8.34 (PA12)
- new net PA2: U8.10 (PA2)
- new net PA4: U8.12 (PA4)
- new net PA5: R46.1, U11.4 (-), U8.13 (PA5)
- new net PA6: R46.2, R47.1, R47.2, U11.1, U8.14 (PA6)
- new net PA7: R45.1, U11.3 (+), U8.15 (PA7)
- new net PA8: U8.30 (PA8)
- new net PC4: U8.16 (PC4)
- new net PC6: U8.29 (PC6)
- new net VREF+: U8.20 (VREF+)
- new net iA+: J3.2 (Pin_2), R44.2, R45.2
- no-connect marks 11 -> 15
Other:
- moved on the sheet: C35, R15, R27, R28

Commit message: schematic
Parts:
- added C47: C, Capacitor_SMD:C_0603_1608Metric, symbol Device:C
- added C48: C, symbol Device:C
- added C49, C50: 100n, Capacitor_SMD:C_0603_1608Metric, symbol Device:C
- added C51, C54: C_Polarized, Capacitor_THT:CP_Radial_D6.3mm_P2.50mm, symbol Device:C_Polarized
- added C52, C55: C, Capacitor_SMD:C_1206_3216Metric, symbol Device:C
- added C53: 10n, Capacitor_SMD:C_0603_1608Metric, symbol Device:C
- added C56: C_Polarized, symbol Device:C_Polarized
- added D8: SM712, Package_TO_SOT_SMD:SOT-23, symbol Diode:SM712_SOT23
- added D9: D_Schottky, Diode_SMD:D_SMF, symbol Device:D_Schottky
- added J15, J16: RS-485, Connector_JST:JST_GH_SM02B-GHS-TB_1x02-1MP_P1.25mm_Horizontal, symbol Connector_Generic_MountingPin:Conn_01x02_MountingPin
- added J6: RS-485, Connector_JST:JST_GH_BM02B-GHS-TBT_1x02-1MP_P1.25mm_Vertical, symbol Connector_Generic_MountingPin:Conn_01x02_MountingPin
- added L2: L, Inductor_SMD:L_Taiyo-Yuden_NR-60xx_HandSoldering, symbol Device:L
- added R51: R, symbol Device:R
- added R52: 100k, symbol Device:R
- added R53, R56, R58: 4.7k, Resistor_SMD:R_0603_1608Metric, symbol Device:R
- added R54, R55: 100, Resistor_SMD:R_0603_1608Metric, symbol Device:R
- added R57: 120, Resistor_SMD:R_0603_1608Metric, symbol Device:R
- added R61: 10k, Resistor_SMD:R_0603_1608Metric, symbol Device:R
- added R62: 1.13k, Resistor_SMD:R_0603_1608Metric, symbol Device:R
- added R63: 10k, symbol Device:R
- added U1: SN75176AD, Package_SO:SOIC-8_3.9x4.9mm_P1.27mm, symbol Interface_UART:SN75176AD
- added U14: TPS5430DDA, Package_SO:TI_SO-PowerPAD-8_ThermalVias, symbol Regulator_Switching:TPS5430DDA
- C15, C16, C17, C18, C19, C38, C39, C41, C46: footprint (none) -> Capacitor_SMD:C_0603_1608Metric
- J3: footprint (none) -> Connector_AMASS:AMASS_XT30U-F_1x02_P5.0mm_Vertical
- R48: value R -> 100k
- R49: now in the parts list
- R50: value R -> 10k; now in the parts list
- R6: footprint (none) -> Resistor_SMD:R_0603_1608Metric
Connections:
- net +3.3VA is gone; now on net +3.3V: C42.1, U7.3 (V+)
- net 1.65Vref is gone; now on net PB1: C40.1, U7.1 (REF)
- net PA10 is gone; now on net Encoder_button: U8.32 (PA10)
- net PA15 is gone; now on net CS: U8.38 (PA15)
- net +24V: now also C51.1, C52.1, U14.7 (VIN)
- net +3.3V: now also R48.1, R50.1, R53.1
- net +5V: now also C49.1, C50.1, R58.2, U1.8 (VCC)
- net GND: now also C47.2, C49.2, C50.2, C51.2, C52.2, C54.2, C55.2, D8.3 (common), D9.2 (A), J15.MP (MountPin), J16.MP (MountPin), J6.MP (MountPin), R51.2, R52.2, R56.1, R62.2, R63.2, U1.5 (GND), U14.6 (GND), U14.9 (GNDPAD); no longer R48.2
- net PA5: now also R51.1
- net PB0: now also R48.2, C47.1, R52.1; no longer R48.1
- net PB1: no longer R50.1, R50.2
- net PB10: now also R54.2
- net PB11: now also R55.1
- net PB14: now also U1.2 (~{RE}), U1.3 (DE)
- net Encoder_button: now reaches R42.1
- net VCC renamed +12V
- net +12V: now also C54.1, C55.1, L2.2, R61.1
- new net: C53.1, U14.1 (BOOT)
- new net: C53.2, D9.1 (K), L2.1, U14.8 (PH)
- new net: R53.2, R55.2, U1.1 (R)
- new net: R61.2, R62.1, U14.4 (VSENSE)
- new net: R54.1, U1.4 (D)
- new net 1.65v: R50.2, R63.1
- new net A+: D8.2 (A2), J15.2 (Pin_2), J16.2 (Pin_2), J6.2 (Pin_2), R57.2, R58.1, U1.6 (A)
- new net B-: D8.1 (A1), J15.1 (Pin_1), J16.1 (Pin_1), J6.1 (Pin_1), R56.2, R57.1, U1.7 (B)
- no-connect marks 15 -> 16
Other:
- moved on the sheet: C22, C25, C27, C28, C29, C30, C34, C42, F2, J8, J9, R10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

Commit message: update sche
Parts:
- removed C51, C54: C_Polarized, Capacitor_THT:CP_Radial_D6.3mm_P2.50mm, symbol Device:C_Polarized
- removed C52, C55: C, Capacitor_SMD:C_1206_3216Metric, symbol Device:C
- removed C53: 10n, Capacitor_SMD:C_0603_1608Metric, symbol Device:C
- removed C56: C_Polarized, symbol Device:C_Polarized
- removed D9: D_Schottky, Diode_SMD:D_SMF, symbol Device:D_Schottky
- removed R63: 10k, symbol Device:R
- removed U14: TPS5430DDA, Package_SO:TI_SO-PowerPAD-8_ThermalVias, symbol Regulator_Switching:TPS5430DDA
- added C51: 22u, Capacitor_SMD:C_1206_3216Metric_Pad1.33x1.80mm_HandSolder, symbol Device:C
- added D10: D_Schottky, Diode_SMD:D_SMF, symbol Device:D_Schottky
- added H1, H2, H3, H4: MountingHole_Pad, MountingHole:MountingHole_2.2mm_M2_Pad_Via, symbol Mechanical:MountingHole_Pad
- added U13: MT3608, Package_TO_SOT_SMD:SOT-23-6, symbol Regulator_Switching:MT3608
- C48: value C -> 22u; footprint (none) -> Inductor_SMD:L_0603_1608Metric
- F1: footprint 0_RM2023:Fuse_1206_1812 -> Fuse:Fuse_1210_3225Metric_Pad1.42x2.65mm_HandSolder
- L2: value L -> 4.7u; footprint Inductor_SMD:L_Taiyo-Yuden_NR-60xx_HandSoldering -> Inductor_SMD:L_0603_1608Metric
- R14, R15, R16, R38, R39, R40, R41, R42, R43, R45, R48, R49, R50, R51, R52: footprint (none) -> Resistor_SMD:R_0603_1608Metric
- R17, R24, R25, R26, R31: footprint (none) -> Resistor_SMD:R_0603_1608Metric_Pad0.98x0.95mm_HandSolder
- R4, R44: footprint (none) -> Resistor_SMD:R_2512_6332Metric
- R6: footprint Resistor_SMD:R_0603_1608Metric -> Resistor_SMD:R_0603_1608Metric_Pad0.98x0.95mm_HandSolder
- R61: value 10k -> 19k
- R62: value 1.13k -> 1k
- SW4: footprint (none) -> Rotary_Encoder:RotaryEncoder_Alps_EC11E-Switch_Vertical_H20mm
- U4: footprint (none) -> Package_SO:MSOP-8_3x3mm_P0.65mm
Connections:
- net +12V: now also C48.1, D10.1 (K); no longer L2.2
- net +3.3V: no longer R50.1
- net +5V: now also L2.1, R50.1, C51.1, U13.5 (IN)
- net GND: now also C48.2, C51.2, H1.1, H2.1, H3.1, H4.1, U13.2 (GND); no longer J4.6 (Pin_6)
- net at R61.2, R62.1: now also U13.3 (FB)
- net 1.65v: no longer names the net of R50.2
- net 1.65v: now also U13.4 (EN)
- new net: D10.2 (A), L2.2, U13.1 (SW)
- new net VSS: J4.6 (Pin_6)
- no-connect marks 16 -> 15
